File: final_Project_2025.kicad_sch (KiCad schematic)
At the start: 20 parts, among them J1 Conn_02x16_Top_Bottom, Q1 TIP42C, Q2 2N2219, Q3 2N2219, Q4 TIP42C, U1 DRV8833PWP, U2 DRV8833PWP, U3 INA219AxD

Commit message: this is the most recent schematic
Parts:
- added SW1: SW_Nidec_CAS-120A1, Button_Switch_SMD:Nidec_Copal_CAS-120A, symbol Switch:SW_Nidec_CAS-120A1
- R3: value R2 -> 2k
Connections:
- net 3.3V: now also U3.1 (A1), U3.5 (VS)
- net Battery: now also U3.8 (IN+); no longer U1.12 (VM), U2.12 (VM)
- net GND: now also U3.2 (A0)
- net Vm1: now reaches U3.7 (IN-)
- net Vm1: now also SW1.3 (A)
- removed net battery: U3.5 (VS), U3.8 (IN+)
- new net Vm: U2.12 (VM)
- new net Vm12: SW1.2 (B)
- new net Vm2: SW1.1 (C), U1.12 (VM)
Other:
- title: Motor control and load switching  -> EEE3088F 2025 Project_Motor driver and Battery charger
- moved on the sheet: R3, U3
